Commit message: Integrate with gazebo
Signed-off-by: Quique Llorente <ellorent@redhat.com>

File: description/robot_core.xacro (robot description, xacro)
@@ -42,3 +42,15 @@
 <xacro:swerve_drive name="front_left" x="1" y="-1" z="-1" r="1"/>
 <xacro:swerve_drive name="rear_left" x="-1" y="-1" z="-1" r="1"/>
+<gazebo reference="base_link">
+    <material>Gazebo/Green</material>
+</gazebo>
+<gazebo reference="chassis">
+    <material>Gazebo/Blue</material>
+</gazebo>
+<gazebo>
+        <plugin name="gazebo_ros_joint_pose_trajectory"
+            filename="libgazebo_ros_joint_pose_trajectory.so">
+            <update_rate>2</update_rate>
+        </plugin>
+    </gazebo>
 </robot>

File: description/robot_swerve_drive.xacro (robot description, xacro)
@@ -21,4 +21,18 @@
             <axis xyz="0 0 -1"/>
         </joint>
+        <gazebo reference="${name}_wheel">
+            <material>Gazebo/Orange</material>
+        </gazebo>
+        <gazebo reference="${name}_steering">
+            <material>Gazebo/Yellow</material>
+        </gazebo>
+    <gazebo>
+        <plugin name="gazebo_ros_joint_state_publisher_${name}"
+            filename="libgazebo_ros_joint_state_publisher.so">
+            <update_rate>20</update_rate>
+            <joint_name>${name}_wheel_joint</joint_name>
+            <joint_name>${name}_steering_joint</joint_name>
+        </plugin>
+    </gazebo>
     </xacro:macro>
 </robot>
