Commit message: reuse swerve drive xacro
Signed-off-by: Quique Llorente <ellorent@redhat.com>

File: description/robot.urdf.xacro (robot description, xacro)
@@ -1,4 +1,6 @@
 <?xml version="1.0"?>
 <robot xmlns:xacro="http://www.ros.org/wiki/xacro"  name="robot">
+    <xacro:include filename="robot_properties.xacro" />
+    <xacro:include filename="robot_swerve_drive.xacro" />
     <xacro:include filename="robot_core.xacro" />
 </robot>

File: description/robot_core.xacro (robot description, xacro)
@@ -24,78 +24,12 @@
         <origin xyz="0 0 0" rpy="0 0 0"/>
         <geometry>
-            <box size="0.280 0.230 0.080"/>
+            <box size="${chassis_length} ${chassis_width} ${chassis_height}"/>
         </geometry>
         <material name="white"/>
     </visual>
 </link>
-<link name="front_right_wheel">
-    <xacro:include filename="robot_wheel.xacro" />
-</link>
-<link name="front_right_steering">
-    <xacro:include filename="robot_steering.xacro" />
-</link>
-<joint name="front_right_steering_joint" type="fixed">
-	<parent link="chassis"/>
-    	<child link="front_right_steering"/>
-	<origin xyz="0.140 0.115 -0.045"/>
-</joint>
-<joint name="front_right_wheel_joint" type="fixed">
-	<parent link="front_right_steering"/>
-    	<child link="front_right_wheel"/>
-	<origin xyz="0 0 -0.025" rpy="-${pi/2} 0 0"/>
-</joint>
-<link name="rear_right_wheel">
-    <xacro:include filename="robot_wheel.xacro" />
-</link>
-<link name="rear_right_steering">
-    <xacro:include filename="robot_steering.xacro" />
-</link>
-<joint name="rear_right_steering_joint" type="fixed">
-	<parent link="chassis"/>
-    	<child link="rear_right_steering"/>
-	<origin xyz="-0.140 0.115 -0.045"/>
-</joint>
-<joint name="rear_right_wheel_joint" type="fixed">
-	<parent link="rear_right_steering"/>
-    	<child link="rear_right_wheel"/>
-	<origin xyz="0 0 -0.025" rpy="-${pi/2} 0 0"/>
-</joint>
-<link name="front_left_wheel">
-    <xacro:include filename="robot_wheel.xacro" />
-</link>
-<link name="front_left_steering">
-    <xacro:include filename="robot_steering.xacro" />
-</link>
-<joint name="front_left_steering_joint" type="fixed">
-	<parent link="chassis"/>
-    	<child link="front_left_steering"/>
-	<origin xyz="0.140 -0.115 -0.045"/>
-</joint>
-<joint name="front_left_wheel_joint" type="fixed">
-	<parent link="front_left_steering"/>
-    	<child link="front_left_wheel"/>
-	<origin xyz="0 0 -0.025" rpy="${pi/2} 0 0"/>
-</joint>
-<joint name="front_left_wheel_join" type="fixed">
-	<parent link="chassis"/>
-    	<child link="front_left_wheel"/>
-    	<origin xyz="0.140 -0.115 -0.065" rpy="${pi/2} 0 0"/>
-	<axis xyz="0 0 1"/>
-</joint>
-<link name="rear_left_wheel">
-    <xacro:include filename="robot_wheel.xacro" />
-</link>
-<link name="rear_left_steering">
-    <xacro:include filename="robot_steering.xacro" />
-</link>
-<joint name="rear_left_steering_joint" type="fixed">
-	<parent link="chassis"/>
-    	<child link="rear_left_steering"/>
-	<origin xyz="-0.140 -0.115 -0.045"/>
-</joint>
-<joint name="rear_left_wheel_joint" type="fixed">
-	<parent link="rear_left_steering"/>
-    	<child link="rear_left_wheel"/>
-	<origin xyz="0 0 -0.025" rpy="${pi/2} 0 0"/>
-</joint>
+<xacro:swerve_drive name="front_right" x="1" y="1" z="-1" r="-1"/>
+<xacro:swerve_drive name="rear_right" x="-1" y="1" z="-1" r="-1"/>
+<xacro:swerve_drive name="front_left" x="1" y="-1" z="-1" r="1"/>
+<xacro:swerve_drive name="rear_left" x="-1" y="-1" z="-1" r="1"/>
 </robot>

Commit message: Add collision and intertial
Signed-off-by: Quique Llorente <ellorent@redhat.com>

File: description/robot.urdf.xacro (robot description, xacro)
@@ -1,4 +1,5 @@
 <?xml version="1.0"?>
 <robot xmlns:xacro="http://www.ros.org/wiki/xacro"  name="robot">
+    <xacro:include filename="inertial_macros.xacro" />
     <xacro:include filename="robot_properties.xacro" />
     <xacro:include filename="robot_swerve_drive.xacro" />

File: description/robot_core.xacro (robot description, xacro)
@@ -28,4 +28,13 @@
         <material name="white"/>
     </visual>
+    <collision>
+        <origin xyz="0 0 0" rpy="0 0 0"/>
+        <geometry>
+            <box size="${chassis_length} ${chassis_width} ${chassis_height}"/>
+        </geometry>
+    </collision>
+    <xacro:inertial_box mass="0.5" x="${chassis_length}" y="${chassis_width}" z="${chassis_height}">
+        <origin xyz="0 0 0" rpy="0 0 0"/>
+    </xacro:inertial_box>
 </link>
 <xacro:swerve_drive name="front_right" x="1" y="1" z="-1" r="-1"/>

File: description/robot_properties.xacro (robot description, xacro)
@@ -4,4 +4,8 @@
     <xacro:property name="chassis_width" value="0.230" />`
     <xacro:property name="chassis_height" value="0.080" />`
+    <xacro:property name="wheel_length" value="0.035" />
+    <xacro:property name="wheel_radius" value="0.020" />
+    <xacro:property name="steering_length" value="0.005" />
+    <xacro:property name="steering_radius" value="0.020" />
     <xacro:property name="steering_joint_x" value="0.140" />`
     <xacro:property name="steering_joint_y" value="0.115" />`

File: description/robot_steering.xacro (robot description, xacro)
@@ -3,7 +3,15 @@
 	<visual>
 	    <geometry>
-		<cylinder length="0.005" radius="0.020" />
+            <cylinder length="${steering_length}" radius="${steering_radius}" />
 	    </geometry>
 	    <material name="blue"/>
-	</visual>
+    </visual>
+    <collision>
+	    <geometry>
+            <cylinder length="${steering_length}" radius="${steering_radius}" />
+	    </geometry>
+    </collision>
+    <xacro:inertial_cylinder mass="0.1" length="${steering_length}" radius="${steering_radius}">
+        <origin xyz="0 0 0" rpy="0 0 0"/>
+    </xacro:inertial_cylinder>
 </link>

File: description/robot_wheel.xacro (robot description, xacro)
@@ -3,7 +3,15 @@
 	<visual>
 	    <geometry>
-		<cylinder length="0.035" radius="0.020" />
+            <cylinder length="${wheel_length}" radius="${wheel_radius}" />
 	    </geometry>
 	    <material name="orange"/>
-	</visual>
+    </visual>
+    <collision>
+	    <geometry>
+            <cylinder length="${wheel_length}" radius="${wheel_radius}" />
+	    </geometry>
+    </collision>
+    <xacro:inertial_cylinder mass="0.1" length="${wheel_length}" radius="${wheel_radius}">
+        <origin xyz="0 0 0" rpy="0 0 0"/>
+    </xacro:inertial_cylinder>
 </link>

Commit message: Integrate ros2_control
Signed-off-by: Quique Llorente <ellorent@redhat.com>

File: description/robot.urdf.xacro (robot description, xacro)
@@ -5,3 +5,5 @@
     <xacro:include filename="robot_swerve_drive.xacro" />
     <xacro:include filename="robot_core.xacro" />
+    <xacro:include filename="ros2_control.xacro"/>
+    <!--xacro:include filename="sim_control.xacro" /-->
 </robot>

File: description/robot_core.xacro (robot description, xacro)
@@ -48,9 +48,3 @@
     <material>Gazebo/Blue</material>
 </gazebo>
-<gazebo>
-        <plugin name="gazebo_ros_joint_pose_trajectory"
-            filename="libgazebo_ros_joint_pose_trajectory.so">
-            <update_rate>2</update_rate>
-        </plugin>
-    </gazebo>
 </robot>

File: description/robot_swerve_drive.xacro (robot description, xacro)
@@ -27,12 +27,26 @@
             <material>Gazebo/Yellow</material>
         </gazebo>
-    <gazebo>
-        <plugin name="gazebo_ros_joint_state_publisher_${name}"
-            filename="libgazebo_ros_joint_state_publisher.so">
-            <update_rate>20</update_rate>
-            <joint_name>${name}_wheel_joint</joint_name>
-            <joint_name>${name}_steering_joint</joint_name>
-        </plugin>
-    </gazebo>
+</xacro:macro>
+    <xacro:macro name="swerve_drive_ros2_control" params="name">
+        <joint name="${name}_wheel_joint">
+            <command_interface name="velocity">
+                <param name="min">-10</param>
+                <param name="max">10</param>
+            </command_interface>
+            <state_interface name="position" />
+            <state_interface name="velocity" />
+        </joint>
+        <joint name="${name}_steering_joint">
+            <command_interface name="position">
+                <param name="min">${-pi/3}</param>
+                <param name="max">${pi/3}</param>
+            </command_interface>
+            <command_interface name="velocity">
+                <param name="min">-10</param>
+                <param name="max">10</param>
+            </command_interface>
+            <state_interface name="position" />
+            <state_interface name="velocity" />
+        </joint>
     </xacro:macro>
 </robot>

Commit message: More work
Signed-off-by: qinqon <quique.llorente@gmail.com>

File: description/robot.urdf.xacro (robot description, xacro)
@@ -1,4 +1,9 @@
 <?xml version="1.0"?>
 <robot xmlns:xacro="http://www.ros.org/wiki/xacro"  name="robot">
+    <xacro:include filename="inertial_macros.xacro" />
+    <xacro:include filename="robot_properties.xacro" />
+    <xacro:include filename="robot_swerve_drive.xacro" />
     <xacro:include filename="robot_core.xacro" />
+    <xacro:include filename="ros2_control.xacro"/>
+    <!--xacro:include filename="sim_control.xacro" /-->
 </robot>

File: description/robot_core.xacro (robot description, xacro)
@@ -24,78 +24,27 @@
         <origin xyz="0 0 0" rpy="0 0 0"/>
         <geometry>
-            <box size="0.280 0.230 0.080"/>
+            <box size="${chassis_length} ${chassis_width} ${chassis_height}"/>
         </geometry>
         <material name="white"/>
     </visual>
+    <collision>
+        <origin xyz="0 0 0" rpy="0 0 0"/>
+        <geometry>
+            <box size="${chassis_length} ${chassis_width} ${chassis_height}"/>
+        </geometry>
+    </collision>
+    <xacro:inertial_box mass="0.5" x="${chassis_length}" y="${chassis_width}" z="${chassis_height}">
+        <origin xyz="0 0 0" rpy="0 0 0"/>
+    </xacro:inertial_box>
 </link>
-<link name="front_right_wheel">
-    <xacro:include filename="robot_wheel.xacro" />
-</link>
-<link name="front_right_steering">
-    <xacro:include filename="robot_steering.xacro" />
-</link>
-<joint name="front_right_steering_joint" type="fixed">
-	<parent link="chassis"/>
-    	<child link="front_right_steering"/>
-	<origin xyz="0.140 0.115 -0.045"/>
-</joint>
-<joint name="front_right_wheel_joint" type="fixed">
-	<parent link="front_right_steering"/>
-    	<child link="front_right_wheel"/>
-	<origin xyz="0 0 -0.025" rpy="-${pi/2} 0 0"/>
-</joint>
-<link name="rear_right_wheel">
-    <xacro:include filename="robot_wheel.xacro" />
-</link>
-<link name="rear_right_steering">
-    <xacro:include filename="robot_steering.xacro" />
-</link>
-<joint name="rear_right_steering_joint" type="fixed">
-	<parent link="chassis"/>
-    	<child link="rear_right_steering"/>
-	<origin xyz="-0.140 0.115 -0.045"/>
-</joint>
-<joint name="rear_right_wheel_joint" type="fixed">
-	<parent link="rear_right_steering"/>
-    	<child link="rear_right_wheel"/>
-	<origin xyz="0 0 -0.025" rpy="-${pi/2} 0 0"/>
-</joint>
-<link name="front_left_wheel">
-    <xacro:include filename="robot_wheel.xacro" />
-</link>
-<link name="front_left_steering">
-    <xacro:include filename="robot_steering.xacro" />
-</link>
-<joint name="front_left_steering_joint" type="fixed">
-	<parent link="chassis"/>
-    	<child link="front_left_steering"/>
-	<origin xyz="0.140 -0.115 -0.045"/>
-</joint>
-<joint name="front_left_wheel_joint" type="fixed">
-	<parent link="front_left_steering"/>
-    	<child link="front_left_wheel"/>
-	<origin xyz="0 0 -0.025" rpy="${pi/2} 0 0"/>
-</joint>
-<joint name="front_left_wheel_join" type="fixed">
-	<parent link="chassis"/>
-    	<child link="front_left_wheel"/>
-    	<origin xyz="0.140 -0.115 -0.065" rpy="${pi/2} 0 0"/>
-	<axis xyz="0 0 1"/>
-</joint>
-<link name="rear_left_wheel">
-    <xacro:include filename="robot_wheel.xacro" />
-</link>
-<link name="rear_left_steering">
-    <xacro:include filename="robot_steering.xacro" />
-</link>
-<joint name="rear_left_steering_joint" type="fixed">
-	<parent link="chassis"/>
-    	<child link="rear_left_steering"/>
-	<origin xyz="-0.140 -0.115 -0.045"/>
-</joint>
-<joint name="rear_left_wheel_joint" type="fixed">
-	<parent link="rear_left_steering"/>
-    	<child link="rear_left_wheel"/>
-	<origin xyz="0 0 -0.025" rpy="${pi/2} 0 0"/>
-</joint>
+<xacro:swerve_drive name="front_right" x="1" y="1" z="-1" r="-1"/>
+<xacro:swerve_drive name="rear_right" x="-1" y="1" z="-1" r="1"/>
+<xacro:swerve_drive name="front_left" x="1" y="-1" z="-1" r="1"/>
+<xacro:swerve_drive name="rear_left" x="-1" y="-1" z="-1" r="1"/>
+<gazebo reference="base_link">
+    <material>Gazebo/Green</material>
+</gazebo>
+<gazebo reference="chassis">
+    <material>Gazebo/Blue</material>
+</gazebo>
 </robot>
