Commit message: Add car like hardware interface
Signed-off-by: qinqon <quique.llorente@gmail.com>

File: description/robot_swerve_drive.xacro (robot description, xacro)
@@ -34,6 +34,6 @@
                 <param name="max">10</param>
             </command_interface>
+            <state_interface name="velocity" />
             <state_interface name="position" />
-            <state_interface name="velocity" />
         </joint>
         <joint name="${name}_steering_joint">
@@ -42,10 +42,5 @@
                 <param name="max">${pi/3}</param>
             </command_interface>
-            <command_interface name="velocity">
-                <param name="min">-10</param>
-                <param name="max">10</param>
-            </command_interface>
             <state_interface name="position" />
-            <state_interface name="velocity" />
         </joint>
     </xacro:macro>

File: description/ros2_control.xacro (robot description, xacro)
@@ -4,37 +4,9 @@
             <hardware>
                 <plugin>robertito/RobertitoDriver</plugin>
-            </hardware>
-            <joint name="front_left_wheel_joint">
-                <command_interface name="velocity">
-                    <param name="min">-10</param>
-                    <param name="max">10</param>
-                </command_interface>
-                <state_interface name="velocity"/>
-                <state_interface name="position"/>
-            </joint>
-            <joint name="front_right_wheel_joint">
-                <command_interface name="velocity">
-                    <param name="min">-10</param>
-                    <param name="max">10</param>
-                </command_interface>
-                <state_interface name="velocity"/>
-                <state_interface name="position"/>
-	    </joint>
-            <joint name="rear_left_wheel_joint">
-                <command_interface name="velocity">
-                    <param name="min">-10</param>
-                    <param name="max">10</param>
-                </command_interface>
-                <state_interface name="velocity"/>
-                <state_interface name="position"/>
-            </joint>
-            <joint name="rear_right_wheel_joint">
-                <command_interface name="velocity">
-                    <param name="min">-10</param>
-                    <param name="max">10</param>
-                </command_interface>
-                <state_interface name="velocity"/>
-                <state_interface name="position"/>
-            </joint>
+	    </hardware>
+	   <xacro:swerve_drive_ros2_control name="front_right"/>
+	   <xacro:swerve_drive_ros2_control name="front_left"/>
+	   <xacro:swerve_drive_ros2_control name="rear_right"/>
+	   <xacro:swerve_drive_ros2_control name="rear_left"/>
         </ros2_control>
 </robot>
